Commit message: Correcciòn a angulos posicion real de robot

File: rapling_description/urdf/prueba.urdf.xacro (robot description, xacro)
@@ -44,4 +44,28 @@
     </collision>
   </link>
+<!-- Enlace "mesa" para limitar el movimiento -->
+<link name="table">
+  <visual>
+    <origin xyz="0 0 0" rpy="0 0 0" />
+    <geometry>
+      <box size="2 2 0.01"/> <!-- Tamaño de la mesa (2x2 metros, grosor 0.01) -->
+    </geometry>
+    <material name="table_color">
+      <color rgba="0.5 0.5 0.5 1"/> <!-- Color gris -->
+    </material>
+  </visual>
+  <collision>
+    <origin xyz="0 0 0" rpy="0 0 0" />
+    <geometry>
+      <box size="2 2 0.01"/>
+    </geometry>
+  </collision>
+</link>
+<!-- Joint fijo para conectar la mesa al mundo -->
+<joint name="table_joint" type="fixed">
+  <parent link="world"/>
+  <child link="table"/>
+  <origin xyz="0 0 -0.066" rpy="0 0 0"/> <!-- Posición de la mesa (en el origen) -->
+</joint>
   <link
     name="Link1">
@@ -119,5 +143,5 @@
         name="">
         <color
-          rgba="0.79216 0.81961 0.93333 1" />
+          rgba="0.6216 0.81961 0.93333 1" />
       </material>
     </visual>
@@ -136,6 +160,6 @@
     type="revolute">
     <origin
-      xyz="0 0 0.035615"
-      rpy="1.5476 -1.553 -1.5478" />
+      xyz="0 0 0.05"
+      rpy="1.5476 -0.0  -1.5478" />
     <parent
       link="Link1" />
@@ -143,8 +167,8 @@
       link="Link_2" />
     <axis
-      xyz="0.0 0.0 -1" />
-    <limit
-      lower="-1.57"
-      upper="1.57"
+      xyz="0.0 0.0 1" />
+    <limit
+      lower="3.14"
+      upper="0.0"
       effort="0"
       velocity="0" />

File: rapling_description/urdf/rapling_ros2_control.xacro (robot description, xacro)
@@ -14,6 +14,6 @@
         <joint name="joint_link_1">
             <command_interface name="position">
-            <param name="min">-${PI / 2}</param>
-            <param name="max">${PI / 2}</param>
+            <param name="min">-${0.0}</param>
+            <param name="max">${PI}</param>
             </command_interface>
             <state_interface name="position"/>
@@ -36,5 +36,5 @@
             <command_interface name="position">
             <param name="min">-${PI / 2}</param>
-            <param name="max">0.0</param>
+            <param name="max">${PI / 2}</param>
             </command_interface>
             <state_interface name="position"/>

Commit message: feat:se actualizo el envio de angulos para las graficas

File: rapling_description/urdf/prueba.urdf.xacro (robot description, xacro)
@@ -271,5 +271,5 @@
         <parent link="base_link" />
         <child link="camera" />
-        <origin  rpy="0 6.28 0" xyz="0.0 0.21 0.40" />
+        <origin  rpy="0 6.28 0" xyz="0.0 0.21 0.34" />
     </joint>
     <link name="camera">

Commit message: agregue task =3 para linea recta

File: rapling_description/urdf/prueba.urdf.xacro (robot description, xacro)
@@ -271,5 +271,5 @@
         <parent link="base_link" />
         <child link="camera" />
-        <origin  rpy="0 6.28 0" xyz="0.0 0.21 0.34" />
+        <origin  rpy="0 6.28 0" xyz="-0.21 0.0 0.34" />
     </joint>
     <link name="camera">

Commit message: actualizaciones de sincronización con robot

File: rapling_description/urdf/prueba.urdf.xacro (robot description, xacro)
@@ -66,5 +66,5 @@
   <parent link="world"/>
   <child link="table"/>
-  <origin xyz="0 0 -0.085" rpy="0 0 0"/> <!-- Posición de la mesa (en el origen) -->
+  <origin xyz="0 0 -0.09" rpy="0 0 0"/> <!-- Posición de la mesa (en el origen) -->
 </joint>
   <link
@@ -271,5 +271,5 @@
         <parent link="base_link" />
         <child link="camera" />
-        <origin  rpy="0 6.28 0" xyz="-0.21 0.0 0.34" />
+        <origin  rpy="0 6.28 0" xyz="-0.21 0.0 0.475" />
     </joint>
     <link name="camera">

Commit message: se agrego un cuadro al mundo y la funciòn de hacer circulo en un goal=4

File: rapling_description/urdf/prueba.urdf.xacro (robot description, xacro)
@@ -282,3 +282,25 @@
         </visual>
     </link>
+<link name="obstacle_1">
+  <visual>
+    <origin xyz="-0.3 -0.2 -0.05" rpy="0 0 0"/>
+    <geometry>
+      <box size="0.1 0.1 0.1"/> <!-- Cubo de 10 cm -->
+    </geometry>
+    <material name="red">
+      <color rgba="1 0 0 1"/> <!-- Color rojo -->
+    </material>
+  </visual>
+  <collision>
+    <origin xyz="-0.3 -0.2 0.05" rpy="0 0 0"/>
+    <geometry>
+      <box size="0.05 0.05 0.05"/>
+    </geometry>
+  </collision>
+</link>
+<joint name="obstacle_1_joint" type="fixed">
+  <parent link="world"/>
+  <child link="obstacle_1"/>
+  <origin xyz="0 0 0" rpy="0 0 0"/>
+</joint>
 </robot>
